Commit message: Controlling Panda robot using moveit through rviz

File: src/multi_panda_moveit_config/config/multi_panda.ros2_control.xacro (robot description, xacro)
@@ -1,5 +1,5 @@
 <?xml version="1.0"?>
 <robot xmlns:xacro="http://www.ros.org/wiki/xacro">
-    <xacro:macro name="multi_panda_ros2_control" params="name initial_positions_file use_sim:=^|false">
+    <xacro:macro name="multi_panda_ros2_control" params="name initial_positions_file use_sim">
         <xacro:property name="initial_positions" value="${xacro.load_yaml(initial_positions_file)['initial_positions']}"/>
         <ros2_control name="${name}" type="system">
